Commit message: Navigation among multiple obstacles - modified xacro fiels to get parameter from launch file

File: uuv_custom_urdf/urdf/box.urdf.xacro (robot description, xacro)
@@ -1,7 +1,10 @@
 <?xml version="1.0" encoding="utf-8"?>
 <robot xmlns:xacro="http://www.ros.org/wiki/xacro" name="box">
-  <xacro:property name="l" value="20" />
-  <xacro:property name="b" value="10" />
-  <xacro:property name="h" value="150" />
+  <xacro:arg name="length" default="20" />
+  <xacro:arg name="breadth" default="10" />
+  <xacro:arg name="height" default="150" />
+  <xacro:property name="l" value="$(arg length)" />
+  <xacro:property name="b" value="$(arg breadth)" />
+  <xacro:property name="h" value="$(arg height)" />
   <!-- Used for fixing robot to Gazebo 'base_link' -->
   <link name="world"/>

File: uuv_custom_urdf/urdf/cylinder.urdf.xacro (robot description, xacro)
@@ -1,6 +1,8 @@
 <?xml version="1.0" encoding="utf-8"?>
 <robot xmlns:xacro="http://www.ros.org/wiki/xacro" name="cylinder">
-  <xacro:property name="r" value="8" />
-  <xacro:property name="h" value="150" />
+  <xacro:arg name="radius" default="1" />
+  <xacro:arg name="height" default="150" />
+  <xacro:property name="r" value="$(arg radius)" />
+  <xacro:property name="h" value="$(arg height)" />
   <!-- Used for fixing robot to Gazebo 'base_link' -->
   <link name="world"/>
